File: eagle/main_borad/main.sch (EAGLE design)
At the start: 1 part

Commit message: mainborad shema - first version
Parts:
- added 1, 2, 3, 4: (no value), pinhead:PINHD-1X9
- added C1, C2: 100nF, eagle-ltspice:CC0201
- added JP1, SUPPLY: (no value), pinhead:PINHD-1X2
- added R1: 10k, eagle-ltspice:RR1206
Connections:
- new net GND: C2.2, SUPPLY.2, U$1.GND@1, U$1.GND@2, U$1.GND@3, U$1.GND@4
- new net N$1: JP1.2, U$1.PDI-CLK/!RESET
- new net N$9: C1.2, JP1.1, R1.2
- new net PA0: 1.5, U$1.PA0(ADC0/AREF)
- new net PA1: 1.4, U$1.PA1(ADC1)
- new net PA2: 1.3, U$1.PA2(ADC2)
- new net PA3: 1.2, U$1.PA3(ADC3)
- new net PA4: 1.1, U$1.PA4(ADC4)
- new net PA5: 2.9, U$1.PA5(ADC5)
- new net PA6: 2.8, U$1.PA6(ADC6)
- new net PA7: 2.7, U$1.PA7/(ADC7/AC0-OUT)
- new net PB0: 2.6, U$1.PB0(ADC8/AREF)
- new net PB1: 2.5, U$1.PB1(ADC9)
- new net PB2: 2.4, U$1.PB2(ADC10/DAC0)
- new net PB3: 2.3, U$1.PB3(ADC11/DAC1)
- new net PC0: 2.2, U$1.PC0(OC0A/SDA)
- new net PC1: 2.1, U$1.PC1(OC0B/XCK0/SCL)
- new net PC2: 3.9, U$1.PC2(OC0C/RXD0)
- new net PC3: 3.8, U$1.PC3(OC0D/TXD0)
- new net PC4: 3.7, U$1.PC4(OC1A/!SS!)
- new net PC5: 3.6, U$1.PC5(OC1B/MOSI/XCK1)
- new net PC6: 3.5, U$1.PC6(MISO/RXD1)
- new net PC7: 3.4, U$1.PC7(SCK/TXD1/CLKO/EVO)
- new net PD0: 3.3, U$1.PD0(OC0A)
- new net PD1: 3.2, U$1.PD1(OC0B/XCK0)
- new net PD2: 3.1, U$1.PD2(OC0C/RXD0)
- new net PD3: 4.9, U$1.PD3(OC0D/TXD0)
- new net PD4: 4.8, U$1.PD4(OC1A/!SS!)
- new net PD5: 4.7, U$1.PD5(OC1B/XCK1/MOSI)
- new net PD6: 4.6, U$1.PD6(RXD1/MISO)
- new net PD7: 4.5, U$1.PD7(TXD1/SCK/CLKO/EVO)
- new net PDI-DATA: 1.9, U$1.PDI-DATA
- new net PE0: 4.4, U$1.PE0(OC0A/SDA)
- new net PE1: 4.3, U$1.PE1(OC0B/XCK0/SCL)
- new net PE2: 4.2, U$1.PE2(OC0C/RXD0)
- new net PE3: 4.1, U$1.PE3(OC0D/TXD0)
- new net PR0: 1.7, U$1.PR0(XTAL2/TOSC1)
- new net PR1: 1.6, U$1.PR1(XTAL1/TOSC1)
- new net RESET: 1.8, C1.1
- new net VCC: C2.1, R1.1, SUPPLY.1, U$1.AVCC, U$1.VCC@1, U$1.VCC@2, U$1.VCC@3
