File: eagle/main_borad/motor_driver.sch (EAGLE design)
At the start: 11 parts, among them Q1 16Mhz, U1 ATMEGA8A-AU

Commit message: mainborad shema - first version
Parts:
- added SUPPLY: (no value), pinhead:PINHD-1X2
Connections:
- net GND: now also SUPPLY.2
- net VCC: now also SUPPLY.1
Other:
- moved on the sheet: 1, 2, 3

Commit message: Druha verze navrhu desek pro rizeni podvozku.
Parts:
- removed 1: (no value), pinhead:PINHD-1X10
- removed 2: (no value), pinhead:PINHD-1X6
- removed 3: (no value), pinhead:PINHD-1X8
- removed C4: 100nF, capacitor-wima:C2,5-3
- removed Q1: 16Mhz, crystal:CRYSTALHC49U-V
- removed RESET_A, SUPPLY: (no value), pinhead:PINHD-1X2
- removed U1: ATMEGA8A-AU, Atmel_By_element14_Batch_1-00:ATMEGA8A-AU
- added C5: 220nF, SparkFun-Capacitors:CAP1206
- added IC1: MEGA8-AI, avr-7:MEGA8-AI
- added JP1, JP2, JP3: (no value), pinhead:PINHD-1X3
- added JP4: (no value), pinhead:PINHD-1X4
- added JP5: (no value), pinhead:PINHD-2X2
- added R2, R3: 5k, eagle-ltspice:RR1206
- added Y1: (no value), SparkFun-FreqCtrl:CRYSTALHC49US
- C1, C2: device capacitor-wima:C2,5-3 -> SparkFun-Capacitors:CAP1206
- C3: value 200nF -> 100nF; device capacitor-wima:C2,5-3 -> SparkFun-Capacitors:CAP1206
- R1: device eagle-ltspice:R -> eagle-ltspice:RR1206
Connections:
- removed net ADC6: 2.5, U1.ADC6
- removed net ADC7: 2.3, U1.ADC7
- removed net AREF: 2.4, U1.AREF
- removed net PB0: 3.1, U1.PB0
- removed net PB1: 3.2, U1.PB1
- removed net PB2: 3.3, U1.PB2
- removed net PB3: 3.4, U1.PB3
- removed net PB4: 3.5, U1.PB4
- removed net PB5: 2.6, U1.PB5
- removed net PC0: 2.2, U1.PC0
- removed net PC1: 2.1, U1.PC1
- removed net PC2: 1.10, U1.PC2
- removed net PC3: 1.9, U1.PC3
- removed net PC4: 1.8, U1.PC4
- removed net PC5: 1.7, U1.PC5
- removed net PD0: 1.5, U1.PD0
- removed net PD1: 1.4, U1.PD1
- removed net PD2: 1.3, U1.PD2
- removed net PD3: 1.2, U1.PD3
- removed net PD4: 1.1, U1.PD4
- removed net PD5: 3.8, U1.PD5
- removed net PD6: 3.7, U1.PD6
- removed net PD7: 3.6, U1.PD7
- removed net ^RESET: C4.2, R1.2, RESET_A.1
- new net INT0: IC1.PD2(INT0), JP2.1
- new net INT1: IC1.PD3(INT1), JP3.1
- new net N$10: IC1.PC4(ADC4/SDA), JP5.1, JP5.2, R2.1
- new net N$12: IC1.PB5(SCK), JP4.4
- new net N$13: IC1.PB4(MISO), JP4.3
- new net N$14: IC1.PB3(MOSI/OC2)
- new net N$15: IC1.PB2(SS/OC1B), JP4.1
- new net N$4: C3.2, IC1.PC6(/RESET), R1.2
- new net N$5: IC1.PD0(RXD), JP1.1
- new net N$6: IC1.PD4(XCK/T0), JP1.3
- new net N$7: JP4.2
- new net N$9: IC1.PC5(ADC5/SCL), JP5.3, JP5.4, R3.1
- net GND: now also C1.1, C2.1, C5.1, IC1.AGND, IC1.GND@1, IC1.GND@2, JP2.2, JP3.2; no longer C1.2, C2.2, C3.2, SUPPLY.2, U1.GND, U1.GND_2, U1.GND_3
- net N$1: now also IC1.PD1(TXD), JP1.2; no longer C1.1, Q1.2, U1.PB6
- net N$2: now also C2.2, IC1.PB7(XTAL2/TOSC2), Y1.1; no longer C2.1, Q1.1, U1.PB7
- net N$3: now also C1.2, IC1.PB6(XTAL1/TOSC1), Y1.2; no longer RESET_A.2, U1.PC6
- net RESET: now also C3.1; no longer 1.6, C4.1
- net VCC: now also C5.2, IC1.AVCC, IC1.VCC@1, IC1.VCC@2, JP2.3, JP3.3, R2.2, R3.2; no longer C3.1, SUPPLY.1, U1.AVCC, U1.VCC, U1.VCC_2
Other:
- moved on the sheet: C1, C2, C3, R1

Commit message: bugfix
Parts:
- added JP6: (no value), pinhead:PINHD-2X2
Connections:
- net GND: now also JP6.3, JP6.4
- net VCC: now also JP6.1, JP6.2
Changed lines of the file:
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@@
 <part name="P+7" library="supply1" deviceset="VCC" device=""/>
 <part name="C5" library="SparkFun-Capacitors" deviceset="CAP" device="1206" value="220nF"/>
+<part name="JP6" library="pinhead" deviceset="PINHD-2X2" device=""/>
+<part name="P+8" library="supply1" deviceset="VCC" device=""/>
+<part name="GND6" library="supply1" deviceset="GND" device=""/>
 </parts>
 <sheets>
@@
 <instance part="P+7" gate="VCC" x="109.22" y="88.9"/>
 <instance part="C5" gate="G$1" x="27.94" y="20.32"/>
+<instance part="JP6" gate="A" x="63.5" y="-22.86"/>
+<instance part="P+8" gate="VCC" x="83.82" y="-20.32" rot="R270"/>
+<instance part="GND6" gate="1" x="81.28" y="-27.94"/>
 </instances>
 <busses>
@@
 <junction x="27.94" y="27.94"/>
 <junction x="27.94" y="30.48"/>
+</segment>
+<segment>
+<pinref part="JP6" gate="A" pin="4"/>
+<wire x1="66.04" y1="-22.86" x2="71.12" y2="-22.86" width="0.1524" layer="91"/>
+<wire x1="71.12" y1="-22.86" x2="81.28" y2="-22.86" width="0.1524" layer="91"/>
+<wire x1="81.28" y1="-22.86" x2="81.28" y2="-25.4" width="0.1524" layer="91"/>
+<wire x1="71.12" y1="-22.86" x2="71.12" y2="-27.94" width="0.1524" layer="91"/>
+<wire x1="71.12" y1="-27.94" x2="53.34" y2="-27.94" width="0.1524" layer="91"/>
+<wire x1="53.34" y1="-27.94" x2="53.34" y2="-22.86" width="0.1524" layer="91"/>
+<pinref part="JP6" gate="A" pin="3"/>
+<wire x1="53.34" y1="-22.86" x2="58.42" y2="-22.86" width="0.1524" layer="91"/>
+<junction x="71.12" y="-22.86"/>
+<pinref part="GND6" gate="1" pin="GND"/>
 </segment>
 </net>
@@
 <junction x="27.94" y="5.08"/>
 </segment>
+<segment>
+<pinref part="JP6" gate="A" pin="1"/>
+<wire x1="58.42" y1="-20.32" x2="53.34" y2="-20.32" width="0.1524" layer="91"/>
+<wire x1="53.34" y1="-20.32" x2="53.34" y2="-15.24" width="0.1524" layer="91"/>
+<wire x1="53.34" y1="-15.24" x2="71.12" y2="-15.24" width="0.1524" layer="91"/>
+<wire x1="71.12" y1="-15.24" x2="71.12" y2="-20.32" width="0.1524" layer="91"/>
+<pinref part="JP6" gate="A" pin="2"/>
+<wire x1="71.12" y1="-20.32" x2="66.04" y2="-20.32" width="0.1524" layer="91"/>
+<wire x1="71.12" y1="-20.32" x2="81.28" y2="-20.32" width="0.1524" layer="91"/>
+<junction x="71.12" y="-20.32"/>
+<pinref part="P+8" gate="VCC" pin="VCC"/>
+</segment>
 </net>

Commit message: motir_driver PCB
Parts:
- added JP7: (no value), pinhead:PINHD-1X1
- added JP8: (no value), pinhead:PINHD-2X2
Connections:
- net GND: now also JP3.3, JP8.3, JP8.4; no longer JP3.2
- net RESET: now also JP7.1
- net VCC: now also JP3.2, JP8.1, JP8.2; no longer JP3.3
Changed lines of the file:
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@@
 <grid distance="0.1" unitdist="inch" unit="inch" style="lines" multiple="1" display="no" altdistance="0.01" altunitdist="inch" altunit="inch"/>
 <layers>
-<layer number="1" name="Top" color="4" fill="1" visible="no" active="no"/>
-<layer number="16" name="Bottom" color="1" fill="1" visible="no" active="no"/>
-<layer number="17" name="Pads" color="2" fill="1" visible="no" active="no"/>
-<layer number="18" name="Vias" color="2" fill="1" visible="no" active="no"/>
-<layer number="19" name="Unrouted" color="6" fill="1" visible="no" active="no"/>
-<layer number="20" name="Dimension" color="15" fill="1" visible="no" active="no"/>
-<layer number="21" name="tPlace" color="7" fill="1" visible="no" active="no"/>
-<layer number="22" name="bPlace" color="7" fill="1" visible="no" active="no"/>
-<layer number="23" name="tOrigins" color="15" fill="1" visible="no" active="no"/>
-<layer number="24" name="bOrigins" color="15" fill="1" visible="no" active="no"/>
-<layer number="25" name="tNames" color="7" fill="1" visible="no" active="no"/>
-<layer number="26" name="bNames" color="7" fill="1" visible="no" active="no"/>
-<layer number="27" name="tValues" color="7" fill="1" visible="no" active="no"/>
-<layer number="28" name="bValues" color="7" fill="1" visible="no" active="no"/>
+<layer number="1" name="Top" color="4" fill="1" visible="yes" active="no"/>
+<layer number="16" name="Bottom" color="1" fill="1" visible="yes" active="no"/>
+<layer number="17" name="Pads" color="2" fill="1" visible="yes" active="no"/>
+<layer number="18" name="Vias" color="2" fill="1" visible="yes" active="no"/>
+<layer number="19" name="Unrouted" color="6" fill="1" visible="yes" active="no"/>
+<layer number="20" name="Dimension" color="15" fill="1" visible="yes" active="no"/>
+<layer number="21" name="tPlace" color="7" fill="1" visible="yes" active="no"/>
+<layer number="22" name="bPlace" color="7" fill="1" visible="yes" active="no"/>
+<layer number="23" name="tOrigins" color="15" fill="1" visible="yes" active="no"/>
+<layer number="24" name="bOrigins" color="15" fill="1" visible="yes" active="no"/>
+<layer number="25" name="tNames" color="7" fill="1" visible="yes" active="no"/>
+<layer number="26" name="bNames" color="7" fill="1" visible="yes" active="no"/>
+<layer number="27" name="tValues" color="7" fill="1" visible="yes" active="no"/>
+<layer number="28" name="bValues" color="7" fill="1" visible="yes" active="no"/>
 <layer number="29" name="tStop" color="7" fill="3" visible="no" active="no"/>
 <layer number="30" name="bStop" color="7" fill="6" visible="no" active="no"/>
@@
 <layer number="35" name="tGlue" color="7" fill="4" visible="no" active="no"/>
 <layer number="36" name="bGlue" color="7" fill="5" visible="no" active="no"/>
-<layer number="37" name="tTest" color="7" fill="1" visible="no" active="no"/>
-<layer number="38" name="bTest" color="7" fill="1" visible="no" active="no"/>
+<layer number="37" name="tTest" color="7" fill="1" visible="yes" active="no"/>
+<layer number="38" name="bTest" color="7" fill="1" visible="yes" active="no"/>
 <layer number="39" name="tKeepout" color="4" fill="11" visible="no" active="no"/>
 <layer number="40" name="bKeepout" color="1" fill="11" visible="no" active="no"/>
@@
 <layer number="44" name="Drills" color="7" fill="1" visible="no" active="no"/>
 <layer number="45" name="Holes" color="7" fill="1" visible="no" active="no"/>
-<layer number="46" name="Milling" color="3" fill="1" visible="no" active="no"/>
-<layer number="47" name="Measures" color="7" fill="1" visible="no" active="no"/>
-<layer number="48" name="Document" color="7" fill="1" visible="no" active="no"/>
-<layer number="49" name="Reference" color="7" fill="1" visible="no" active="no"/>
-<layer number="50" name="dxf" color="7" fill="1" visible="no" active="no"/>
-<layer number="51" name="tDocu" color="7" fill="1" visible="no" active="no"/>
-<layer number="52" name="bDocu" color="7" fill="1" visible="no" active="no"/>
-<layer number="53" name="tGND_GNDA" color="7" fill="9" visible="no" active="no"/>
-<layer number="54" name="bGND_GNDA" color="1" fill="9" visible="no" active="no"/>
-<layer number="56" name="wert" color="7" fill="1" visible="no" active="no"/>
-<layer number="57" name="tCAD" color="7" fill="1" visible="no" active="no"/>
+<layer number="46" name="Milling" color="3" fill="1" visible="yes" active="no"/>
+<layer number="47" name="Measures" color="7" fill="1" visible="yes" active="no"/>
+<layer number="48" name="Document" color="7" fill="1" visible="yes" active="no"/>
+<layer number="49" name="Reference" color="7" fill="1" visible="yes" active="no"/>
+<layer number="50" name="dxf" color="7" fill="1" visible="yes" active="no"/>
+<layer number="51" name="tDocu" color="7" fill="1" visible="yes" active="no"/>
+<layer number="52" name="bDocu" color="7" fill="1" visible="yes" active="no"/>
+<layer number="53" name="tGND_GNDA" color="7" fill="9" visible="yes" active="no"/>
+<layer number="54" name="bGND_GNDA" color="1" fill="9" visible="yes" active="no"/>
+<layer number="56" name="wert" color="7" fill="1" visible="yes" active="no"/>
+<layer number="57" name="tCAD" color="7" fill="1" visible="yes" active="no"/>
 <layer number="90" name="Modules" color="5" fill="1" visible="yes" active="yes"/>
 <layer number="91" name="Nets" color="2" fill="1" visible="yes" active="yes"/>
@@
 <part name="P+8" library="supply1" deviceset="VCC" device=""/>
 <part name="GND6" library="supply1" deviceset="GND" device=""/>
+<part name="JP7" library="pinhead" deviceset="PINHD-1X1" device=""/>
+<part name="JP8" library="pinhead" deviceset="PINHD-2X2" device=""/>
+<part name="P+9" library="supply1" deviceset="VCC" device=""/>
+<part name="GND7" library="supply1" deviceset="GND" device=""/>
 </parts>
 <sheets>
@@
 <instance part="P+8" gate="VCC" x="83.82" y="-20.32" rot="R270"/>
 <instance part="GND6" gate="1" x="81.28" y="-27.94"/>
+<instance part="JP7" gate="G$1" x="5.08" y="68.58" rot="R180"/>
+<instance part="JP8" gate="A" x="63.5" y="-45.72"/>
+<instance part="P+9" gate="VCC" x="83.82" y="-43.18" rot="R270"/>
+<instance part="GND7" gate="1" x="81.28" y="-50.8"/>
 </instances>
 <busses>
@@
 <pinref part="JP2" gate="A" pin="2"/>
 <wire x1="160.02" y1="40.64" x2="144.78" y2="40.64" width="0.1524" layer="91"/>
-<wire x1="144.78" y1="40.64" x2="144.78" y2="25.4" width="0.1524" layer="91"/>
-<pinref part="JP3" gate="A" pin="2"/>
-<wire x1="144.78" y1="25.4" x2="144.78" y2="17.78" width="0.1524" layer="91"/>
-<wire x1="160.02" y1="25.4" x2="144.78" y2="25.4" width="0.1524" layer="91"/>
-<junction x="144.78" y="25.4"/>
+<wire x1="144.78" y1="40.64" x2="144.78" y2="22.86" width="0.1524" layer="91"/>
 <pinref part="GND5" gate="1" pin="GND"/>
+<pinref part="JP3" gate="A" pin="3"/>
+<wire x1="144.78" y1="22.86" x2="144.78" y2="17.78" width="0.1524" layer="91"/>
+<wire x1="144.78" y1="22.86" x2="160.02" y2="22.86" width="0.1524" layer="91"/>
+<junction x="144.78" y="22.86"/>
 </segment>
 <segment>
@@
 <pinref part="GND6" gate="1" pin="GND"/>
 </segment>
+<segment>
+<pinref part="JP8" gate="A" pin="4"/>
+<wire x1="66.04" y1="-45.72" x2="71.12" y2="-45.72" width="0.1524" layer="91"/>
+<wire x1="71.12" y1="-45.72" x2="81.28" y2="-45.72" width="0.1524" layer="91"/>
+<wire x1="81.28" y1="-45.72" x2="81.28" y2="-48.26" width="0.1524" layer="91"/>
+<wire x1="71.12" y1="-45.72" x2="71.12" y2="-50.8" width="0.1524" layer="91"/>
+<wire x1="71.12" y1="-50.8" x2="53.34" y2="-50.8" width="0.1524" layer="91"/>
+<wire x1="53.34" y1="-50.8" x2="53.34" y2="-45.72" width="0.1524" layer="91"/>
+<pinref part="JP8" gate="A" pin="3"/>
+<wire x1="53.34" y1="-45.72" x2="58.42" y2="-45.72" width="0.1524" layer="91"/>
+<junction x="71.12" y="-45.72"/>
+<pinref part="GND7" gate="1" pin="GND"/>
+</segment>
 </net>
 <net name="VCC" class="0">
@@
 <pinref part="JP2" gate="A" pin="3"/>
 <wire x1="160.02" y1="38.1" x2="147.32" y2="38.1" width="0.1524" layer="91"/>
-<wire x1="147.32" y1="38.1" x2="147.32" y2="22.86" width="0.1524" layer="91"/>
-<pinref part="JP3" gate="A" pin="3"/>
-<wire x1="147.32" y1="22.86" x2="147.32" y2="20.32" width="0.1524" layer="91"/>
-<wire x1="160.02" y1="22.86" x2="147.32" y2="22.86" width="0.1524" layer="91"/>
-<junction x="147.32" y="22.86"/>
+<wire x1="147.32" y1="38.1" x2="147.32" y2="25.4" width="0.1524" layer="91"/>
 <pinref part="P+5" gate="VCC" pin="VCC"/>
+<pinref part="JP3" gate="A" pin="2"/>
+<wire x1="147.32" y1="25.4" x2="147.32" y2="20.32" width="0.1524" layer="91"/>
+<wire x1="160.02" y1="25.4" x2="147.32" y2="25.4" width="0.1524" layer="91"/>
+<junction x="147.32" y="25.4"/>
 </segment>
 <segment>
@@
 <pinref part="P+8" gate="VCC" pin="VCC"/>
 </segment>
+<segment>
+<pinref part="JP8" gate="A" pin="1"/>
+<wire x1="58.42" y1="-43.18" x2="53.34" y2="-43.18" width="0.1524" layer="91"/>
+<wire x1="53.34" y1="-43.18" x2="53.34" y2="-38.1" width="0.1524" layer="91"/>
+<wire x1="53.34" y1="-38.1" x2="71.12" y2="-38.1" width="0.1524" layer="91"/>
+<wire x1="71.12" y1="-38.1" x2="71.12" y2="-43.18" width="0.1524" layer="91"/>
+<pinref part="JP8" gate="A" pin="2"/>
+<wire x1="71.12" y1="-43.18" x2="66.04" y2="-43.18" width="0.1524" layer="91"/>
+<wire x1="71.12" y1="-43.18" x2="81.28" y2="-43.18" width="0.1524" layer="91"/>
+<junction x="71.12" y="-43.18"/>
+<pinref part="P+9" gate="VCC" pin="VCC"/>
+</segment>
 </net>
 <net name="N$9" class="0">
@@
 <pinref part="C3" gate="G$1" pin="1"/>
 <wire x1="17.78" y1="68.58" x2="7.62" y2="68.58" width="0.1524" layer="91"/>
-<label x="7.62" y="68.58" size="1.778" layer="95" rot="R180" xref="yes"/>
-</segment>
-</net>
+<pinref part="JP7" gate="G$1" pin="1"/>
+</segment>
+</net>

Commit message: PCB ver. 4.0
Parts:
- Y1: device SparkFun-FreqCtrl:CRYSTALHC49US -> SparkFun-FreqCtrl:CRYSTALSMD
Changed lines of the file:
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@@
 <part name="GND3" library="supply1" deviceset="GND" device=""/>
 <part name="P+3" library="supply1" deviceset="VCC" device=""/>
-<part name="Y1" library="SparkFun-FreqCtrl" deviceset="CRYSTAL" device="HC49US"/>
+<part name="Y1" library="SparkFun-FreqCtrl" deviceset="CRYSTAL" device="SMD"/>
 <part name="C1" library="SparkFun-Capacitors" deviceset="CAP" device="1206" value="220pF"/>
 <part name="C2" library="SparkFun-Capacitors" deviceset="CAP" device="1206" value="220pF"/>

Commit message: PCB layout 6.0
Parts:
- C5: device SparkFun-Capacitors:CAP1206 -> SparkFun-Capacitors:CAP0805
Changed lines of the file:
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@@
 <part name="P+6" library="supply1" deviceset="VCC" device=""/>
 <part name="P+7" library="supply1" deviceset="VCC" device=""/>
-<part name="C5" library="SparkFun-Capacitors" deviceset="CAP" device="1206" value="220nF"/>
+<part name="C5" library="SparkFun-Capacitors" deviceset="CAP" device="0805" value="220nF"/>
 <part name="JP6" library="pinhead" deviceset="PINHD-2X2" device=""/>
 <part name="P+8" library="supply1" deviceset="VCC" device=""/>
