File: eagle/switch_boards/motor12v.sch (EAGLE design)
At the start: 9 parts

Commit message: Motor switch board ver.  2.0
Parts:
- added OUT4, OUT5, OUT6, SWITCH: (no value), con-ptr500:AK500/2
- C1: value (none) -> 100uF
- IN12V, OUT1, OUT2, OUT3: device con-ptr500:AK500/2-H -> con-ptr500:AK500/2
Connections:
- removed net OUT_GND: C1.-, D2.A, D3.A, OUT1-1.KL, OUT2-1.KL, OUT3-1.KL, R1.2
- new net EN21: C1.+, D3.C, F1.1
- new net IN12V: D3.A, SWITCH-1.KL
- net +12V: now also IN12V-1.KL, SWITCH-2.KL; no longer C1.+, F1.1, IN12V-2.KL
- net GND: now also C1.-, D2.A, IN12V-2.KL, OUT1-1.KL, OUT2-1.KL, OUT3-1.KL, OUT4-1.KL, OUT5-1.KL, OUT6-1.KL, R1.2; no longer D3.C, IN12V-1.KL
- net OUT_+12V: now also OUT4-2.KL, OUT5-2.KL, OUT6-2.KL
Other:
- moved on the sheet: D3, IN12V-1, IN12V-2
Changed lines of the file:
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@@
 <?xml version="1.0" encoding="utf-8"?>
 <!DOCTYPE eagle SYSTEM "eagle.dtd">
-<eagle version="7.1.0">
+<eagle version="7.2.0">
 <drawing>
 <settings>
@@
 </classes>
 <parts>
-<part name="OUT1" library="con-ptr500" deviceset="AK500/2-H" device=""/>
-<part name="C1" library="resistor" deviceset="CPOL-EU" device="E3.5-8"/>
-<part name="IN12V" library="con-ptr500" deviceset="AK500/2-H" device=""/>
+<part name="OUT1" library="con-ptr500" deviceset="AK500/2" device=""/>
+<part name="C1" library="resistor" deviceset="CPOL-EU" device="E3.5-8" value="100uF"/>
+<part name="IN12V" library="con-ptr500" deviceset="AK500/2" device=""/>
 <part name="GND1" library="supply1" deviceset="GND" device=""/>
 <part name="P+1" library="supply1" deviceset="+12V" device=""/>
 <part name="GND2" library="supply1" deviceset="GND" device=""/>
-<part name="P+2" library="supply1" deviceset="+12V" device=""/>
 <part name="D2" library="diode" deviceset="1N4148" device="DO35-10"/>
 <part name="D3" library="diode" deviceset="1N5400" device=""/>
 <part name="F1" library="fuse" deviceset="FUSE" device="BLANK_5X20MM"/>
-<part name="OUT2" library="con-ptr500" deviceset="AK500/2-H" device=""/>
-<part name="OUT3" library="con-ptr500" deviceset="AK500/2-H" device=""/>
+<part name="OUT2" library="con-ptr500" deviceset="AK500/2" device=""/>
+<part name="OUT3" library="con-ptr500" deviceset="AK500/2" device=""/>
 <part name="R1" library="varistor" deviceset="S2220" device=""/>
+<part name="OUT4" library="con-ptr500" deviceset="AK500/2" device=""/>
+<part name="OUT5" library="con-ptr500" deviceset="AK500/2" device=""/>
+<part name="OUT6" library="con-ptr500" deviceset="AK500/2" device=""/>
+<part name="SWITCH" library="con-ptr500" deviceset="AK500/2" device=""/>
+<part name="P+3" library="supply1" deviceset="+12V" device=""/>
 </parts>
 <sheets>
@@
 <instance part="OUT1" gate="-2" x="88.9" y="33.02"/>
 <instance part="C1" gate="G$1" x="119.38" y="66.04" rot="R180"/>
-<instance part="IN12V" gate="-1" x="81.28" y="71.12"/>
-<instance part="IN12V" gate="-2" x="81.28" y="66.04"/>
+<instance part="IN12V" gate="-1" x="81.28" y="66.04"/>
+<instance part="IN12V" gate="-2" x="81.28" y="71.12"/>
 <instance part="GND1" gate="1" x="88.9" y="76.2" rot="R180"/>
 <instance part="P+1" gate="1" x="88.9" y="60.96" rot="R180"/>
 <instance part="GND2" gate="1" x="106.68" y="76.2" rot="R270"/>
-<instance part="P+2" gate="1" x="106.68" y="60.96" rot="R90"/>
 <instance part="D2" gate="G$1" x="134.62" y="68.58" smashed="yes" rot="R270">
 <attribute name="NAME" x="129.54" y="63.9826" size="1.778" layer="95"/>
 <attribute name="VALUE" x="134.3914" y="78.74" size="1.778" layer="96" rot="R90"/>
 </instance>
-<instance part="D3" gate="1" x="114.3" y="76.2" smashed="yes" rot="R180">
-<attribute name="NAME" x="114.3" y="73.1774" size="1.778" layer="95" rot="R180"/>
-<attribute name="VALUE" x="119.38" y="81.0514" size="1.778" layer="96" rot="R180"/>
+<instance part="D3" gate="1" x="111.76" y="60.96" smashed="yes">
+<attribute name="NAME" x="109.22" y="56.3626" size="1.778" layer="95"/>
+<attribute name="VALUE" x="106.68" y="63.7286" size="1.778" layer="96"/>
 </instance>
 <instance part="F1" gate="G$1" x="127" y="60.96"/>
@@
 <attribute name="VALUE" x="147.955" y="67.31" size="1.778" layer="96" rot="R90"/>
 </instance>
+<instance part="OUT4" gate="-1" x="129.54" y="38.1"/>
+<instance part="OUT4" gate="-2" x="129.54" y="33.02"/>
+<instance part="OUT5" gate="-1" x="129.54" y="25.4"/>
+<instance part="OUT5" gate="-2" x="129.54" y="20.32"/>
+<instance part="OUT6" gate="-1" x="129.54" y="12.7"/>
+<instance part="OUT6" gate="-2" x="129.54" y="7.62"/>
+<instance part="SWITCH" gate="-1" x="53.34" y="71.12"/>
+<instance part="SWITCH" gate="-2" x="53.34" y="66.04"/>
+<instance part="P+3" gate="1" x="60.96" y="60.96" rot="R180"/>
 </instances>
 <busses>
@@
 <net name="GND" class="0">
 <segment>
-<pinref part="IN12V" gate="-1" pin="KL"/>
 <pinref part="GND1" gate="1" pin="GND"/>
 <wire x1="86.36" y1="71.12" x2="88.9" y2="71.12" width="0.1524" layer="91"/>
 <wire x1="88.9" y1="71.12" x2="88.9" y2="73.66" width="0.1524" layer="91"/>
-</segment>
-<segment>
-<pinref part="GND2" gate="1" pin="GND"/>
-<wire x1="111.76" y1="76.2" x2="109.22" y2="76.2" width="0.1524" layer="91"/>
-<pinref part="D3" gate="1" pin="C"/>
-</segment>
-</net>
-<net name="+12V" class="0">
-<segment>
 <pinref part="IN12V" gate="-2" pin="KL"/>
-<pinref part="P+1" gate="1" pin="+12V"/>
-<wire x1="86.36" y1="66.04" x2="88.9" y2="66.04" width="0.1524" layer="91"/>
-<wire x1="88.9" y1="66.04" x2="88.9" y2="63.5" width="0.1524" layer="91"/>
-</segment>
-<segment>
-<pinref part="P+2" gate="1" pin="+12V"/>
-<pinref part="C1" gate="G$1" pin="+"/>
-<wire x1="119.38" y1="63.5" x2="119.38" y2="60.96" width="0.1524" layer="91"/>
-<wire x1="109.22" y1="60.96" x2="119.38" y2="60.96" width="0.1524" layer="91"/>
-<pinref part="F1" gate="G$1" pin="1"/>
-<wire x1="119.38" y1="60.96" x2="121.92" y2="60.96" width="0.1524" layer="91"/>
-<junction x="119.38" y="60.96"/>
-</segment>
-</net>
-<net name="OUT_GND" class="0">
-<segment>
-<wire x1="116.84" y1="76.2" x2="119.38" y2="76.2" width="0.1524" layer="91"/>
+</segment>
+<segment>
 <pinref part="C1" gate="G$1" pin="-"/>
 <wire x1="119.38" y1="76.2" x2="119.38" y2="71.12" width="0.1524" layer="91"/>
 <pinref part="D2" gate="G$1" pin="A"/>
 <wire x1="134.62" y1="71.12" x2="134.62" y2="76.2" width="0.1524" layer="91"/>
-<pinref part="D3" gate="1" pin="A"/>
 <junction x="134.62" y="76.2"/>
 <wire x1="119.38" y1="76.2" x2="134.62" y2="76.2" width="0.1524" layer="91"/>
 <label x="152.4" y="76.2" size="1.778" layer="95"/>
 <wire x1="134.62" y1="76.2" x2="142.24" y2="76.2" width="0.1524" layer="91"/>
-<junction x="119.38" y="76.2"/>
 <pinref part="R1" gate="1" pin="2"/>
 <wire x1="142.24" y1="76.2" x2="157.48" y2="76.2" width="0.1524" layer="91"/>
 <wire x1="142.24" y1="73.66" x2="142.24" y2="76.2" width="0.1524" layer="91"/>
 <junction x="142.24" y="76.2"/>
+<pinref part="GND2" gate="1" pin="GND"/>
+<wire x1="109.22" y1="76.2" x2="119.38" y2="76.2" width="0.1524" layer="91"/>
+<junction x="119.38" y="76.2"/>
 </segment>
 <segment>
@@
 <wire x1="93.98" y1="12.7" x2="101.6" y2="12.7" width="0.1524" layer="91"/>
 <label x="99.06" y="12.7" size="1.778" layer="95"/>
+</segment>
+<segment>
+<pinref part="OUT4" gate="-1" pin="KL"/>
+<wire x1="134.62" y1="38.1" x2="142.24" y2="38.1" width="0.1524" layer="91"/>
+<label x="139.7" y="38.1" size="1.778" layer="95"/>
+</segment>
+<segment>
+<pinref part="OUT5" gate="-1" pin="KL"/>
+<wire x1="134.62" y1="25.4" x2="142.24" y2="25.4" width="0.1524" layer="91"/>
+<label x="139.7" y="25.4" size="1.778" layer="95"/>
+</segment>
+<segment>
+<pinref part="OUT6" gate="-1" pin="KL"/>
+<wire x1="134.62" y1="12.7" x2="142.24" y2="12.7" width="0.1524" layer="91"/>
+<label x="139.7" y="12.7" size="1.778" layer="95"/>
+</segment>
+</net>
+<net name="+12V" class="0">
+<segment>
+<pinref part="P+1" gate="1" pin="+12V"/>
+<wire x1="88.9" y1="66.04" x2="88.9" y2="63.5" width="0.1524" layer="91"/>
+<pinref part="IN12V" gate="-1" pin="KL"/>
+<wire x1="88.9" y1="66.04" x2="86.36" y2="66.04" width="0.1524" layer="91"/>
+</segment>
+<segment>
+<pinref part="SWITCH" gate="-2" pin="KL"/>
+<pinref part="P+3" gate="1" pin="+12V"/>
+<wire x1="58.42" y1="66.04" x2="60.96" y2="66.04" width="0.1524" layer="91"/>
+<wire x1="60.96" y1="66.04" x2="60.96" y2="63.5" width="0.1524" layer="91"/>
 </segment>
 </net>
@@
 <label x="99.06" y="7.62" size="1.778" layer="95"/>
 </segment>
-</net>
+<segment>
+<pinref part="OUT4" gate="-2" pin="KL"/>
+<wire x1="134.62" y1="33.02" x2="142.24" y2="33.02" width="0.1524" layer="91"/>
+<label x="139.7" y="33.02" size="1.778" layer="95"/>
+</segment>
+<segment>
+<pinref part="OUT5" gate="-2" pin="KL"/>
+<wire x1="134.62" y1="20.32" x2="142.24" y2="20.32" width="0.1524" layer="91"/>
+<label x="139.7" y="20.32" size="1.778" layer="95"/>
+</segment>
+<segment>
+<pinref part="OUT6" gate="-2" pin="KL"/>
+<wire x1="134.62" y1="7.62" x2="142.24" y2="7.62" width="0.1524" layer="91"/>
+<label x="139.7" y="7.62" size="1.778" layer="95"/>
+</segment>
+</net>
+<net name="IN12V" class="0">
+<segment>
+<pinref part="SWITCH" gate="-1" pin="KL"/>
+<wire x1="58.42" y1="71.12" x2="60.96" y2="71.12" width="0.1524" layer="91"/>
+<wire x1="60.96" y1="71.12" x2="60.96" y2="78.74" width="0.1524" layer="91"/>
+<label x="60.96" y="76.2" size="1.778" layer="95" rot="R90"/>
+</segment>
+<segment>
+<label x="101.6" y="60.96" size="1.778" layer="95"/>
+<pinref part="D3" gate="1" pin="A"/>
+<wire x1="104.14" y1="60.96" x2="109.22" y2="60.96" width="0.1524" layer="91"/>
+</segment>
+</net>
+<net name="EN21" class="0">
+<segment>
+<pinref part="C1" gate="G$1" pin="+"/>
+<wire x1="119.38" y1="63.5" x2="119.38" y2="60.96" width="0.1524" layer="91"/>
+<pinref part="F1" gate="G$1" pin="1"/>
+<wire x1="119.38" y1="60.96" x2="121.92" y2="60.96" width="0.1524" layer="91"/>
+<pinref part="D3" gate="1" pin="C"/>
+<wire x1="119.38" y1="60.96" x2="114.3" y2="60.96" width="0.1524" layer="91"/>
+<junction x="119.38" y="60.96"/>
+</segment>
+</net>
